File: pcb/qs-80-sbc.kicad_sch (KiCad schematic)
At the start: 56 parts, among them J1 BUS, J2 USB_B, J3 DE9_Socket, J4 Atmel-JTAG-10, J5 KEYBOARD, J6 MOUSE, SW1 ON, SW2 RESET, SW3 NMI, U1 Z84C0020, U2 CY62256-70PC, U22 MAX232, U3 ATmega328P-P, U4 SST39SF010, U5 ATF1504AS-xJx44, U6 TL16C2550PFBR, U7 74HC273, U8 VERA MJ, Y1 14.7456 MHz, Y2 16MHz

Commit message: Adding 74HC138 for port mapping
Parts:
- added U9: 74HC138, symbol 74xx:74HC138
Connections:
- net A14: now also U5.6 (I/O); no longer U5.29 (I/O)
- net A15: now also U5.8 (I/O)
- net A2: no longer U5.6 (I/O)
- net A3: no longer U5.8 (I/O)
- net A4: no longer U5.9 (I/O)
- net A5: now also U9.1 (A0); no longer U5.11 (I/O/PD1)
- net A6: now also U9.2 (A1); no longer U5.12 (I/O)
- net A7: now also U9.3 (A2); no longer U5.14 (I/O)
- net BANK_LATCH: now also U9.12 (~{Y3}); no longer U5.31 (I/O)
- net D0: no longer U5.33 (I/O)
- net D1: no longer U5.34 (I/O)
- net D2: no longer U5.36 (I/O)
- net D3: no longer U5.37 (I/O)
- net D4: no longer U5.39 (I/O)
- net GND: now also U9.8 (GND)
- net VCC: now also U9.16 (VCC), U9.6 (E2)
- net ~{IORQ}: now also U9.5 (~{E1})
- net ~{M1}: now also U9.4 (~{E0})
- net ~{RAM_CS}: now also U5.24 (I/O); no longer U5.25 (I/O/PD2)
- net ~{RES}: no longer U7.1 (~{Mr})
- net ~{ROM_CS}: now also U5.25 (I/O/PD2); no longer U5.26 (I/O)
- net ~{UART_CSA}: now also U9.14 (~{Y1}); no longer U5.27 (I/O)
- net ~{UART_CSB}: now also U9.13 (~{Y2}); no longer U5.28 (I/O)
- net ~{VERA_CS}: now also U9.15 (~{Y0}); no longer U5.24 (I/O)
- new net ~{BANKCLR}: U5.26 (I/O), U7.1 (~{Mr})
- no-connect marks 31 -> 35
Other:
- moved on the sheet: D10, R5

Commit message: Tuning I/O ports
Parts:
- removed U2: CY62256-70PC, Package_DIP:DIP-28_W15.24mm, symbol Memory_RAM:CY62256-70PC
- removed U7: 74HC273, Package_DIP:DIP-20_W7.62mm_Socket, symbol 74xx:74HC273
- removed U9: 74HC138, symbol 74xx:74HC138
- added U2: AS6C1008-xxP, Package_DIP:DIP-32_W15.24mm, symbol Memory_RAM:AS6C1008-xxP
Connections:
- net ROMS3 is gone; now on net ROMS1: U4.3 (A15)
- net ROMS4 is gone; now on net ROMS2: U4.2 (A16)
- net ~{BANKCLR} is gone; now on net A5: U5.26 (I/O)
- net A0: now also U2.12 (A0)
- net A1: now also U2.11 (A1)
- net A10: now also U2.23 (A10)
- net A11: now also U2.25 (A11)
- net A12: now also U4.4 (A12), U2.4 (A12); no longer U5.4 (I/O)
- net A13: now also U4.28 (A13), U2.28 (A13); no longer U5.5 (I/O)
- net A14: now also U5.4 (I/O); no longer U5.6 (I/O)
- net A15: now also U5.5 (I/O); no longer U5.43 (I/GCLK1), U5.8 (I/O)
- net A2: now also U2.10 (A2)
- net A3: now also U2.9 (A3)
- net A4: now also U2.8 (A4)
- net A5: now also U2.7 (A5)
- net A6: now also U5.43 (I/GCLK1), U2.6 (A6)
- net A7: now also U5.28 (I/O), U2.5 (A7)
- net A8: now also U2.27 (A8)
- net A9: now also U2.26 (A9)
- net D0: now also U5.11 (I/O/PD1), U2.13 (DQ0)
- net D1: now also U5.12 (I/O), U2.14 (DQ1)
- net D2: now also U5.33 (I/O), U2.15 (DQ2)
- net D3: now also U5.34 (I/O), U2.17 (DQ3)
- net D4: now also U2.18 (DQ4)
- net D5: now also U2.19 (DQ5)
- net D6: now also U2.20 (DQ6)
- net D7: now also U2.21 (DQ7)
- net GND: now also U2.16 (GND)
- net RAMS0: now also U5.36 (I/O), U2.3 (A14)
- net RAMS1: now also U5.37 (I/O), U2.31 (A15)
- net RAMS2: now also U5.39 (I/O), U2.2 (A16)
- net ROMS0: now also U4.29 (A14), U5.6 (I/O); no longer U4.4 (A12)
- net ROMS1: now also U5.8 (I/O); no longer U4.28 (A13)
- net ROMS2: now also U5.9 (I/O); no longer U4.29 (A14)
- net VCC: now also U2.30 (CS2/CE2), U2.32 (VCC)
- net ~{RAM_CS}: now also U2.22 (~{CS1}/~{CE1})
- net ~{RD}: now also U2.24 (~{OE})
- net ~{UART_CSA}: now also U5.31 (I/O)
- net ~{UART_CSB}: now also U5.29 (I/O)
- net ~{VERA_CS}: now also U5.27 (I/O)
- net ~{WR}: now also U2.29 (~{WE})
- no-connect marks 35 -> 32

Commit message: Initial routing
Parts:
- removed C9: 0.1uF, Capacitor_THT:C_Disc_D5.0mm_W2.5mm_P5.00mm, symbol Device:C
- removed R2, R6, R7: 10k, Resistor_THT:R_Axial_DIN0207_L6.3mm_D2.5mm_P7.62mm_Horizontal, symbol Device:R_Small
- added RN1: 10k, Resistor_THT:R_Array_SIP9, symbol Device:R_Network08
- U1: footprint Package_DIP:DIP-40_W15.24mm -> Package_DIP:DIP-40_W15.24mm_Socket
- U2: footprint Package_DIP:DIP-32_W15.24mm -> Package_DIP:DIP-32_W15.24mm_Socket
- U3: footprint Package_DIP:DIP-28_W7.62mm -> Package_DIP:DIP-28_W7.62mm_Socket
Connections:
- net A14: now also U5.40 (I/O); no longer U5.4 (I/O)
- net A15: now also U5.39 (I/O); no longer U5.5 (I/O)
- net A5: now also U5.24 (I/O); no longer U5.26 (I/O)
- net A6: now also U5.21 (I/O); no longer U5.43 (I/GCLK1)
- net A7: now also U5.19 (I/O); no longer U5.28 (I/O)
- net CLK: now also U5.43 (I/GCLK1)
- net D0: now also U5.37 (I/O); no longer U5.11 (I/O/PD1)
- net D1: now also U5.36 (I/O); no longer U5.12 (I/O)
- net D2: now also U5.34 (I/O); no longer U5.33 (I/O)
- net D3: now also U5.33 (I/O); no longer U5.34 (I/O)
- net RAMS0: now also U5.17 (I/O); no longer U5.36 (I/O)
- net RAMS1: now also U5.16 (I/O); no longer U5.37 (I/O)
- net RAMS2: now also U5.14 (I/O); no longer U5.39 (I/O)
- net ROMS0: now also U5.12 (I/O); no longer U5.6 (I/O)
- net ROMS1: now also U5.11 (I/O/PD1); no longer U5.8 (I/O)
- net VCC: now also RN1.1 (common)
- net VERA_INT: now also U5.6 (I/O); no longer U5.40 (I/O)
- net ~{HALT}: now also RN1.5 (R4)
- net ~{INT}: now also U5.31 (I/O), RN1.7 (R6); no longer U5.21 (I/O)
- net ~{IORQ}: now also U5.27 (I/O); no longer U5.17 (I/O)
- net ~{M1}: now also U5.28 (I/O); no longer U5.20 (I/O)
- net ~{MRQ}: now also U5.29 (I/O); no longer U5.16 (I/O)
- net ~{NMI}: now also RN1.6 (R5)
- net ~{RAM_CS}: now also U5.18 (I/O); no longer U5.24 (I/O)
- net ~{RD}: now also U5.25 (I/O/PD2); no longer U5.18 (I/O)
- net ~{ROM_CS}: now also U5.20 (I/O); no longer U5.25 (I/O/PD2)
- net ~{UART_CSA}: now also U5.4 (I/O); no longer U5.31 (I/O)
- net ~{UART_CSB}: now also U5.5 (I/O); no longer U5.29 (I/O)
- net ~{VERA_CS}: now also U5.8 (I/O); no longer U5.27 (I/O)
- net ~{WAIT}: now also RN1.4 (R3)
- net ~{WR}: now also U5.26 (I/O); no longer U5.19 (I/O)
- net at U1.23 (~{BUSACK}): now also RN1.8 (R7)
- net at U1.25 (~{BUSREQ}): now also RN1.9 (R8)
- net at R3.2: now also J2.SH (Shield); no longer J2.5 (Shield)
- no-connect marks 32 -> 31

Commit message: Completing routing phase 1
Parts:
- added H1, H2, H3, H4: MountingHole, MountingHole:MountingHole_3.2mm_M3_DIN965_Pad, symbol Mechanical:MountingHole
- U2: value AS6C1008-xxP -> AS6C1008
- U5: value ATF1504AS-xJx44 -> ATF1504AS
Connections:
- net GND: now also J3.SH (shield), J5.SH (shield), J6.SH (shield)

Commit message: Adding reset diode
Parts:
- added D1: 1N4148, Diode_THT:D_DO-35_SOD27_P7.62mm_Horizontal, symbol Diode:1N4148
- added R2: 22, Resistor_THT:R_Axial_DIN0207_L6.3mm_D2.5mm_P7.62mm_Horizontal, symbol Device:R
- C15: value 220uF -> 47uF
Connections:
- net BTN_RES: now also D1.1 (K)
- net CLK: now also R2.2; no longer Y1.8 (OUT)
- net at RN2.9 (R8.2), U3.1 (~{RESET}/PC6): now also D1.2 (A)
- new net: R2.1, Y1.8 (OUT)
Other:
- moved on the sheet: RN2H
