File: pcb/qs-80-sbc.kicad_pcb (KiCad board)
At the start: 2 copper layers, 124.5 x 124.5 mm, 56 parts, among them J1 BUS, J2 USB_B, J3 DE9_Socket, J4 Atmel-JTAG-10, J5 KEYBOARD, J6 MOUSE, SW1 ON, SW2 RESET, SW3 NMI, U1 Z84C0020, U2 CY62256-70PC, U22 MAX232, U3 ATmega328P-P, U4 SST39SF010, U5 ATF1504AS-xJx44, U6 TL16C2550PFBR, U7 74HC273, U8 VERA MJ, Y1 14.7456 MHz, Y2 16MHz

Commit message: Initial routing
Parts:
- removed C9: 0.1uF, Capacitor_THT:C_Disc_D5.0mm_W2.5mm_P5.00mm
- removed R2, R6, R7: 10k, Resistor_THT:R_Axial_DIN0207_L6.3mm_D2.5mm_P7.62mm_Horizontal
- removed U7: 74HC273, Package_DIP:DIP-20_W7.62mm_Socket
- added RN1: 10k, Resistor_THT:R_Array_SIP9, F.Cu at (102.0, 131.8)
- U1: footprint Package_DIP:DIP-40_W15.24mm -> Package_DIP:DIP-40_W15.24mm_Socket
- U2: value CY62256-70PC -> AS6C1008-xxP; footprint Package_DIP:DIP-28_W15.24mm -> Package_DIP:DIP-32_W15.24mm_Socket
- U3: footprint Package_DIP:DIP-28_W7.62mm -> Package_DIP:DIP-28_W7.62mm_Socket
- moved C27 182.1 mm to (25.4, 47.7), turned to -90 degrees
- moved C11 157.6 mm to (70.5, 39.6), turned to -90 degrees
- moved C14 145.7 mm to (74.3, 44.6), turned to 90 degrees
- moved C12 145.0 mm to (108.0, 40.6)
- moved C6 144.5 mm to (36.8, 81.3), turned to 180 degrees
- moved C17 142.5 mm to (66.7, 58.7), turned to -90 degrees
- moved R10 138.8 mm to (60.3, 45.9), turned to 90 degrees
- moved R11 136.8 mm to (83.2, 45.9), turned to 90 degrees
- moved R8 136.7 mm to (65.4, 38.3), turned to -90 degrees
- moved R9 129.9 mm to (78.1, 45.9), turned to 90 degrees
- moved R3 127.1 mm to (134.0, 24.1), turned to -90 degrees
- moved C10 125.0 mm to (87.0, 63.7), turned to 90 degrees
- moved C1 123.7 mm to (70.5, 58.7), turned to -90 degrees
- moved C8 121.3 mm to (61.6, 81.3), turned to 180 degrees
- moved C13 111.6 mm to (110.6, 58.4)
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Connections:
- J2 pad SH: (no net) -> Net-(J2-Shield)
- U1 pad 23: unconnected-(U1-~{BUSACK}-Pad23) -> Net-(RN1-R7)
- U1 pad 25: unconnected-(U1-~{BUSREQ}-Pad25) -> Net-(RN1-R8)
- U2 pad 1: RAMS2 -> unconnected-(U2-NC-Pad1)
- U2 pad 10: A0 -> A2
- U2 pad 11: D0 -> A1
- U2 pad 12: D1 -> A0
- U2 pad 13: D2 -> D0
- U2 pad 14: GND -> D1
- U2 pad 15: D3 -> D2
- U2 pad 16: D4 -> GND
- U2 pad 17: D5 -> D3
- U2 pad 18: D6 -> D4
- U2 pad 19: D7 -> D5
- U2 pad 2: RAMS0 -> RAMS2
- U2 pad 20: ~{RAM_CS} -> D6
- U2 pad 21: A10 -> D7
- U2 pad 22: ~{RD} -> ~{RAM_CS}
- U2 pad 23: A11 -> A10
- U2 pad 24: A9 -> ~{RD}
- U2 pad 25: A8 -> A11
- U2 pad 26: RAMS1 -> A9
- U2 pad 27: ~{WR} -> A8
- U2 pad 28: VCC -> A13
- U2 pad 3: A7 -> RAMS0
- U2 pad 4: A6 -> A12
- U2 pad 5: A5 -> A7
- U2 pad 6: A4 -> A6
- U2 pad 7: A3 -> A5
- U2 pad 8: A2 -> A4
- U2 pad 9: A1 -> A3
- U4 pad 2: ROMS4 -> ROMS2
- U4 pad 28: ROMS1 -> A13
- U4 pad 29: ROMS2 -> ROMS0
- U4 pad 3: ROMS3 -> ROMS1
- U4 pad 4: ROMS0 -> A12
- U5 pad 11: A5 -> ROMS1
- U5 pad 12: A6 -> ROMS0
- U5 pad 14: A7 -> RAMS2
- U5 pad 16: ~{MRQ} -> RAMS1
- U5 pad 17: ~{IORQ} -> RAMS0
- U5 pad 18: ~{RD} -> ~{RAM_CS}
- U5 pad 19: ~{WR} -> A7
- U5 pad 20: ~{M1} -> ~{ROM_CS}
- U5 pad 21: ~{INT} -> A6
- U5 pad 24: ~{VERA_CS} -> A5
- U5 pad 25: ~{RAM_CS} -> ~{RD}
- U5 pad 26: ~{ROM_CS} -> ~{WR}
- U5 pad 27: ~{UART_CSA} -> ~{IORQ}
- U5 pad 28: ~{UART_CSB} -> ~{M1}
- U5 pad 29: A14 -> ~{MRQ}
- U5 pad 31: BANK_LATCH -> ~{INT}
- U5 pad 33: D0 -> D3
- U5 pad 34: D1 -> D2
- U5 pad 36: D2 -> D1
- U5 pad 37: D3 -> D0
- U5 pad 39: D4 -> A15
- U5 pad 4: A12 -> ~{UART_CSA}
- U5 pad 40: VERA_INT -> A14
- U5 pad 43: A15 -> CLK
- U5 pad 5: A13 -> ~{UART_CSB}
- U5 pad 6: A2 -> VERA_INT
- U5 pad 8: A3 -> ~{VERA_CS}
- U5 pad 9: A4 -> ROMS2
Routing:
- net GND: track 0.00 -> 1194.8 mm, vias 0 -> 13
- net VCC: track 0.00 -> 1068.4 mm, vias 0 -> 18
- net D4: track 0.00 -> 291.4 mm, vias 0 -> 9
- net ~{RD}: track 0.00 -> 274.2 mm, vias 0 -> 10
- net D6: track 0.00 -> 269.1 mm, vias 0 -> 9
- net D0: track 0.00 -> 269.0 mm, vias 0 -> 8
- net D2: track 0.00 -> 268.3 mm, vias 0 -> 9
- net D7: track 0.00 -> 259.0 mm, vias 0 -> 6
- net D1: track 0.00 -> 247.9 mm, vias 0 -> 7
- net ~{WR}: track 0.00 -> 235.0 mm, vias 0 -> 6
- net D3: track 0.00 -> 233.5 mm, vias 0 -> 6
- net D5: track 0.00 -> 227.9 mm, vias 0 -> 7
- net A0: track 0.00 -> 219.8 mm, vias 0 -> 7
- net ~{HALT}: track 0.00 -> 206.7 mm, vias 0 -> 2
- net ~{NMI}: track 0.00 -> 198.7 mm, vias 0 -> 3
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
Commit message: Completing routing phase 1
Parts:
- added H1: MountingHole, MountingHole:MountingHole_3.2mm_M3_DIN965_Pad, F.Cu at (20.5, 21.8)
- added H2: MountingHole, MountingHole:MountingHole_3.2mm_M3_DIN965_Pad, F.Cu at (137.0, 21.8)
- added H3: MountingHole, MountingHole:MountingHole_3.2mm_M3_DIN965_Pad, F.Cu at (20.5, 138.2)
- added H4: MountingHole, MountingHole:MountingHole_3.2mm_M3_DIN965_Pad, F.Cu at (137.0, 138.2)
- U2: value AS6C1008-xxP -> AS6C1008
- U5: value ATF1504AS-xJx44 -> ATF1504AS
- moved R3 11.4 mm to (134.0, 35.6), turned to 90 degrees
- moved R10 0.22 mm to (60.3, 45.7)
- moved R11 0.22 mm to (83.2, 45.7)
- moved R8 0.22 mm to (65.4, 38.1)
- moved R9 0.22 mm to (78.1, 45.7)
- moved C1 0.10 mm to (70.5, 58.8)
- moved C10 0.10 mm to (87.0, 63.8)
- moved C17 0.10 mm to (66.7, 58.8)
Connections:
- J3 pad SH: (no net) -> GND
- J5 pad SH: (no net) -> GND
- J6 pad SH: (no net) -> GND
Routing:
- net VCC: track 1068.4 -> 767.4 mm
- net GND: track 1194.8 -> 1022.8 mm
- net Net-(J2-Shield): track 110.2 -> 29.9 mm, vias 1 -> 0
- net ~{RD}: track 274.2 -> 272.5 mm, vias 10 -> 9
- net D0: track 269.0 -> 268.6 mm, vias 8 -> 7
- net D1: track 247.9 -> 247.5 mm, vias 7 -> 6
- net ~{RTSB}: vias 4 -> 3
- net ~{CTSB}: vias 4 -> 3
- added copper zone on F.Cu, net GND
- added copper zone on B.Cu, net VCC
Other:
- outline, holes or cut-outs redrawn

Commit message: Adding reset diode
Parts:
- added D1: 1N4148, Diode_THT:D_DO-35_SOD27_P7.62mm_Horizontal, F.Cu at (85.1, 34.5)
- added R2: 22, Resistor_THT:R_Axial_DIN0207_L6.3mm_D2.5mm_P7.62mm_Horizontal, F.Cu at (120.7, 60.3)
- C15: value 220uF -> 47uF
Connections:
- Y1 pad 8: CLK -> Net-(Y1-OUT)
Routing:
- net CLK: track 150.5 -> 166.8 mm
- net Net-(D1-A): track 50.0 -> 61.7 mm
- net BTN_RES: track 135.2 -> 144.3 mm
- net Net-(Y1-OUT): track 0.00 -> 4.32 mm
- net MS_DATA: track 12.2 -> 13.5 mm
Other:
- board text added: "5V power only no data"
- board text added: "KEYBOARD"
- board text added: "MOUSE"

Commit message: Storing
Parts:
- moved C5 1.00 mm to (126.0, 96.6)
Routing:
- net GND: track 1022.8 -> 1056.7 mm, vias 13 -> 19
Other:
- board text added: "A0"
- board text added: "A1"
- board text added: "A10"
- board text added: "A11"
- board text added: "A12"
- board text added: "A13"
- board text added: "A14"
- board text added: "A15"
- board text added: "A2"
- board text added: "A3"
- board text added: "A4"
- board text added: "A5"
- board text added: "A6"
- board text added: "A7"
- board text added: "A8"
- board text added: "A9"
- board text added: "CLK"
- board text added: "D0"
- board text added: "D1"
- board text added: "D2"
- board text added: "D3"
- board text added: "D4"
- board text added: "D5"
- board text added: "D6"
- board text added: "D7"
- board text added: "GND"
- board text added: "QuickSilver - 80 Single Board Z80-based computer"
- board text added: "VCC"
- board text added: "v1"
- board text added: "~{HALT}"
- board text added: "~{INT}"
- board text added: "~{IORQ}"
- board text added: "~{M1}"
- board text added: "~{MREQ}"
- board text added: "~{NMI}"
- board text added: "~{RD}"
- board text added: "~{RESET}"
- board text added: "~{WAIT}"
- board text added: "~{WR}"
